Commit message: Where Am I, with teleoperation package

File: my_robot/urdf/my_robot.xacro (robot description, xacro)
@@ -39,7 +39,7 @@
     <origin xyz="0 0 0" rpy="0 0 0" />
     <parent link="robot_footprint"/>
-    <child link="chassis" />
-  </joint>
-  <link name="chassis">
+    <child link="base_link" />
+  </joint>
+  <link name="base_link">
     <pose>0 0 0.1 0 0 0</pose>
     <inertial>

Commit message: feat: Proj5. Map my World The project incorporates the RTABMAP to generate a Db file.

File: my_robot/urdf/my_robot.xacro (robot description, xacro)
@@ -191,5 +191,5 @@
   </link>
   <joint name="camera_joint" type="fixed">
-    <origin xyz="0.2 0.0 0.0" rpy="0.0 0.0 0.0"/>
+    <origin xyz="0.15 0 ${2*box_z}" rpy="0.0 0.0 0.0"/>
     <parent link="robot_footprint"/>
     <child link="camera"/>
@@ -224,3 +224,11 @@
     <axis xyz="0.0 1.0 0.0"/>
   </joint>
+<!--Optical camera RGBD -->
+<joint name="camera_optical_joint" type="fixed">
+    <origin xyz="0 0 0" rpy="-1.5707 0 -1.5707"/>
+    <parent link="camera"/>
+    <child link="camera_link_optical"/>
+  </joint>
+  <link name="camera_link_optical">
+  </link>
 </robot>
